Commit message: Update LiDAR mount transform and add slow-drive test

File: src/vidalia_bringup/urdf/amiga_min.urdf (robot description, URDF)
Before this commit: robot amiga_min, 2 links, 1 joints
Joints:
- joint base_to_velodyne: origin xyz=1.130 0.0 0.80 rpy=0 0 0 -> xyz=0.959 0.0 0.699 rpy=0 0 0
