Commit message: Set LiDAR forward x offset to 0.85 m (1 ft ahead of front tires)
New mount is 1 ft (0.30 m) forward of the front-tire centres. base_link is the
robot-footprint centre, and the front tires sit ~0.55 m ahead of it (half the
~1.10 m wheelbase per amiga_min.urdf), so base_link->velodyne x = 0.55 + 0.30 =
0.85 m (was 0.959 m). Updated URDF, all three TF launch files, and the two ROS
node param defaults/docstrings. Half-wheelbase (0.55 m) is the one assumption —
flagged in-file to confirm. Native brain stack is unaffected (doesn't use x).

Co-Authored-By: Claude Sonnet 5 <noreply@anthropic.com>
Claude-Session: https://claude.ai/code/session_01RYuc67Meajai11QPmDXdYB

File: src/vidalia_bringup/urdf/amiga_min.urdf (robot description, URDF)
Before this commit: robot amiga_min, 2 links, 1 joints
Joints:
- joint base_to_velodyne: origin xyz=0.959 0.0 0.699 rpy=0 0 0 -> xyz=0.85 0.0 0.800 rpy=0 0 0

Commit message: LiDAR raised to ~0.99 m: mount-height update, calibration tooling, onion re-validation
The VLP-16 was raised from 0.80 m to ~0.98-1.00 m (mount otherwise unchanged).

- LIDAR_MOUNT_HEIGHT 0.80 -> 0.99 (provisional until the box calibration)
  in obstacle_filter, ROS 2 bridge TF, URDF, static-TF launch files, ROS node
  defaults; viz_perception imports the constant.
- row_follow.py --lidar-height: per-run override (set_mount_height rebinds
  every importing module), recorded in the run manifest.
- diag_pitch_rings.py prints the tilt/height to use; diag_birdseye.py reports
  the implied mount height from the tilt sweep and checks a --box-height.
- Onion bed mode re-validated at 0.99 m in the ray-cast sim (still passes at
  0.80 m): count-first bed-axis cue selection (height-variance cue dragged a
  mature-canopy axis 5 deg at U-turn re-entry), comb ratio 1.4 lock / 1.3 hold,
  trimmed furrow-line fit, absolute 5 cm floor on the bed-end quarter check.
- Tall-canopy limit moves from ~0.63 m to ~0.82 m plants.
- Calibration procedure documented in CLAUDE.md; tests for the override,
  cue selection and the poisoned-baseline bed-end case.

Co-Authored-By: Claude Opus 5.5 <noreply@anthropic.com>
Claude-Session: https://claude.ai/code/session_01RYuc67Meajai11QPmDXdYB

File: src/vidalia_bringup/urdf/amiga_min.urdf (robot description, URDF)
Before this commit: robot amiga_min, 2 links, 1 joints
Joints:
- joint base_to_velodyne: origin xyz=0.85 0.0 0.800 rpy=0 0 0 -> xyz=0.85 0.0 0.990 rpy=0 0 0

Commit message: Calibrate the raised LiDAR mount: 1.035 m, 15.7 deg tilt, 0.9 deg yaw
Flat warehouse floor (2026-10-29): raw ring fit 15.7-15.8 deg / 1.036 m,
floor -0.005 m at 1.03 m, 0.40 m box reads 0.40 m, box azimuth -0.9 deg.

- obstacle_filter: LIDAR_MOUNT_HEIGHT = 1.035 plus LIDAR_TILT_DEG = 15.7 and
  LIDAR_YAW_DEG = 0.9, now the defaults of row_follow, slam_mapper,
  diag_birdseye, the SLAM engine and the onion simulator; ROS bridge, URDF
  and launch z = 1.035.
- Bed-end cut/axis-hold/latch arm only once the far bed has shown relief
  since the reset: under a tall canopy at the steeper tilt a false latch
  capped confidence at 0.3 and a near-quarter axis search ran away 10 deg.
- diag_sensor_model: drop the stale "driver table is wrong" message.
- Docs and CHANGELOG: calibration values, flat-ground requirement, new sim
  results (all stages <= 2.4 cm bias) and tall-canopy limits.

Co-Authored-By: Claude Opus 5.5 <noreply@anthropic.com>
Claude-Session: https://claude.ai/code/session_01RYuc67Meajai11QPmDXdYB

File: src/vidalia_bringup/urdf/amiga_min.urdf (robot description, URDF)
Before this commit: robot amiga_min, 2 links, 1 joints
Joints:
- joint base_to_velodyne: origin xyz=0.85 0.0 0.990 rpy=0 0 0 -> xyz=0.85 0.0 1.035 rpy=0 0 0
